File: PdlSerialAdapter.brd (EAGLE design)
At the start: 46 x 17.8 mm, 12 parts, among them X2 PN61729-S

Commit message: New version
Parts:
- added C4: 100nF, rcl:C050-030X075
- added JP1: POWER, pinhead:1X02
- added LED1: TX, led:LED3MM
- added LED2: RX, led:LED3MM
- added R1, R2: 1k, rcl:0207/2V
- C1: value (none) -> 22pF; device rcl:C050-030X075 -> rcl:C025-025X050
- C2: value (none) -> 22pF
- C3: value (none) -> 10nF; device rcl:C025-025X050 -> rcl:C050-030X075
- Q1: value (none) -> 12MHz
- moved C1 10.6 mm to (28.6, 15.2), turned to 90 degrees
- moved C2 8.64 mm to (28.6, 10.2)
- moved Q1 3.18 mm to (33.7, 12.7)
- moved RX 2.54 mm to (49.5, 14.0)
- moved TX 2.54 mm to (49.5, 11.4)
- moved U$1 2.01 mm to (41.3, 12.1)
- moved C3 1.90 mm to (23.5, 12.7), turned to 270 degrees
Connections:
- new net N$3: 5V.1, JP1.1
- new net N$6: LED1.A, R1.1
- new net N$7: LED2.A, R2.1
- net +5V: now also C4.2, JP1.2, R1.2, R2.2; no longer 5V.1
- net GND: now also C4.1
- net N$1: now also C1.2; no longer C2.2
- net N$2: now also C2.2; no longer C3.2
- net N$4: now also C3.2; no longer C1.2
- net N$5: now also LED1.K
- net RX: now also LED2.K
Routing:
- net N$5: track 13.4 -> 35.4 mm
- net RX: track 11.8 -> 31.1 mm, vias 2 -> 0
- net +5V: track 48.7 -> 65.3 mm
- net N$6: track 0.00 -> 14.3 mm
- net N$3: track 0.00 -> 13.4 mm
- net D-: track 23.8 -> 31.1 mm, vias 0 -> 1
- net N$4: track 22.2 -> 16.1 mm
- net N$2: track 16.0 -> 11.6 mm
- net D+: track 26.3 -> 30.3 mm, vias 0 -> 1
- net N$7: track 0.00 -> 3.70 mm
- net GND: track 62.7 -> 59.2 mm, vias 0 -> 1
- net N$1: track 20.5 -> 17.5 mm, vias 1 -> 0
Other:
- board text added: "PdLSerialAdapter v1.1"
- board text removed: "PdLSerialAdapter v1.0"
