File: PdlSerialAdapter.sch (EAGLE design)
At the start: 12 parts, among them X2 PN61729-S

Commit message: New version
Parts:
- added C4: 100nF, rcl:C-EU050-030X075
- added JP1: POWER, pinhead:PINHD-1X2
- added LED1: TX, led:LED3MM
- added LED2: RX, led:LED3MM
- added R1, R2: 1k, rcl:R-EU_0207/2V
- C1: value (none) -> 22pF; device rcl:C-EU050-030X075 -> rcl:C-EU025-025X050
- C2: value (none) -> 22pF
- C3: value (none) -> 10nF; device rcl:C-EU025-025X050 -> rcl:C-EU050-030X075
- Q1: value (none) -> 12MHz
Connections:
- new net N$3: 5V.P, JP1.1
- new net N$6: LED1.A, R1.1
- new net N$7: LED2.A, R2.1
- net +5V: now also C4.2, JP1.2, R1.2, R2.2; no longer 5V.P
- net GND: now also C4.1
- net N$1: now also C1.2; no longer C2.2
- net N$2: now also C2.2; no longer C3.2
- net N$4: now also C3.2; no longer C1.2
- net N$5: now also LED1.C
- net RX: now also LED2.C
Other:
- moved on the sheet: C1, C2, C3
